File: MP3Player.kicad_sch (KiCad schematic)
At the start: 8 parts, among them J1 3.5mm TRRS, SW1 Switch_Tactile_ESwitch, SW2 Switch_Tactile_ESwitch, SW3 Switch_Tactile_ESwitch, SW4 Switch_Tactile_ESwitch, U1 DFR0299, U2 DM-OLED096-636

Commit message: general update
Parts:
- added BT2: BH-18650-A1AJ005, JLCImport:BH-18650-A1AJ005, symbol JLCImport:BH-18650-A1AJ005
- added M1: TP4056Module, Library:TP4056Module, symbol Library:root_0_TP4056Module_Schlib1.SchLib
- SWDown1: renamed from SW4; footprint PCM_fab:Button_ESwitch_TL3315NF100Q_4.5x4.5mm -> PCM_SparkFun-Switch:Push_SMD_6.2x6.2mm
- SWLeft1: renamed from SW2; footprint PCM_fab:Button_ESwitch_TL3315NF100Q_4.5x4.5mm -> PCM_SparkFun-Switch:Push_SMD_6.2x6.2mm
- SWRight1: renamed from SW3; footprint PCM_fab:Button_ESwitch_TL3315NF100Q_4.5x4.5mm -> PCM_SparkFun-Switch:Push_SMD_6.2x6.2mm
- SWUp1: renamed from SW1; footprint PCM_fab:Button_ESwitch_TL3315NF100Q_4.5x4.5mm -> PCM_SparkFun-Switch:Push_SMD_6.2x6.2mm
Connections:
- net GND: now also U2.1 (GND); no longer A1.GND1 (GND)
- net at SWUp1.1, SWUp1.2: now also A1.D3 (D3_INT1); no longer A1.D2 (D2_INT0)
- net at SWUp1.3, SWUp1.4: no longer A1.D3 (D3_INT1)
- net at SWLeft1.1, SWLeft1.2: now also A1.D5; no longer A1.D4
- net at SWLeft1.3, SWLeft1.4: no longer A1.D5
- net at SWRight1.1, SWRight1.2: now also A1.D7; no longer A1.D6
- net at SWRight1.3, SWRight1.4: no longer A1.D7
- net at SWDown1.1, SWDown1.2: now also A1.D9; no longer A1.D8
- net at SWDown1.3, SWDown1.4: now also A1.GND2 (GND); no longer A1.D9
- net at A1.VIN: now also M1.3 (OUT+)
- new net: A1.GND1 (GND), M1.6 (OUT-)
- new net: BT2.1, M1.5 (B-)
- new net: BT2.2, M1.4 (B+)
Other:
- moved on the sheet: SWDown1, SWLeft1, SWRight1, SWUp1

Commit message: e
Connections:
- net at A1.D0 (D0/RX): no longer U1.3 (TX)
- net at A1.D1 (D1/TX): no longer U1.2 (RX)
- net at A1.D2 (D2_INT0): now also U1.2 (RX)
- net at A1.D4: now also U1.3 (TX)
- net at A1.GND2 (GND), SWDown1.3, SWDown1.4: now also SWLeft1.3, SWLeft1.4, SWRight1.3, SWRight1.4, SWUp1.3, SWUp1.4
Changed lines of the file:
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@@
 	(paper "A4")
+	(junction
+		(at 203.2 116.84)
+		(diameter 0)
+		(color 0 0 0 0)
+	)
 	(junction
 		(at 137.16 142.24)
@@
 		(color 0 0 0 0)
 	)
+	(junction
+		(at 203.2 111.76)
+		(diameter 0)
+		(color 0 0 0 0)
+	)
+	(junction
+		(at 203.2 121.92)
+		(diameter 0)
+		(color 0 0 0 0)
+	)
 	(wire
 		(pts
@@
 	(wire
 		(pts
+			(xy 142.24 55.88) (xy 142.24 58.42)
+		)
+		(stroke
+			(width 0)
+			(type default)
+		)
+	)
+	(wire
+		(pts
 			(xy 190.5 106.68) (xy 193.04 106.68)
 		)
@@
 	(wire
 		(pts
+			(xy 194.31 109.22) (xy 194.31 54.61)
+		)
+		(stroke
+			(width 0)
+			(type default)
+		)
+	)
+	(wire
+		(pts
 			(xy 137.16 119.38) (xy 137.16 142.24)
 		)
@@
 	(wire
 		(pts
+			(xy 190.5 55.88) (xy 142.24 55.88)
+		)
+		(stroke
+			(width 0)
+			(type default)
+		)
+	)
+	(wire
+		(pts
 			(xy 133.35 118.11) (xy 138.43 118.11)
 		)
@@
 	(wire
 		(pts
+			(xy 194.31 54.61) (xy 139.7 54.61)
+		)
+		(stroke
+			(width 0)
+			(type default)
+		)
+	)
+	(wire
+		(pts
 			(xy 92.71 142.24) (xy 137.16 142.24)
 		)
@@
 	(wire
 		(pts
+			(xy 190.5 104.14) (xy 190.5 55.88)
+		)
+		(stroke
+			(width 0)
+			(type default)
+		)
+	)
+	(wire
+		(pts
 			(xy 125.73 168.91) (xy 130.81 168.91)
 		)
@@
 	(wire
 		(pts
-			(xy 116.84 53.34) (xy 116.84 106.68)
-		)
-		(stroke
-			(width 0)
-			(type default)
-		)
-	)
-	(wire
-		(pts
 			(xy 127 58.42) (xy 92.71 58.42)
 		)
@@
 	(wire
 		(pts
-			(xy 142.24 58.42) (xy 142.24 53.34)
-		)
-		(stroke
-			(width 0)
-			(type default)
-		)
-	)
-	(wire
-		(pts
-			(xy 139.7 52.07) (xy 115.57 52.07)
+			(xy 139.7 54.61) (xy 139.7 58.42)
 		)
 		(stroke
@@
 	(wire
 		(pts
-			(xy 142.24 53.34) (xy 116.84 53.34)
-		)
-		(stroke
-			(width 0)
-			(type default)
-		)
-	)
-	(wire
-		(pts
 			(xy 190.5 121.92) (xy 193.04 121.92)
 		)
@@
 	(wire
 		(pts
+			(xy 203.2 106.68) (xy 203.2 111.76)
+		)
+		(stroke
+			(width 0)
+			(type default)
+		)
+	)
+	(wire
+		(pts
 			(xy 130.81 124.46) (xy 133.35 124.46)
 		)
@@
 	(wire
 		(pts
-			(xy 139.7 58.42) (xy 139.7 52.07)
+			(xy 190.5 109.22) (xy 194.31 109.22)
 		)
 		(stroke
@@
 	(wire
 		(pts
-			(xy 115.57 104.14) (xy 139.7 104.14)
+			(xy 203.2 116.84) (xy 203.2 121.92)
 		)
 		(stroke
@@
 	(wire
 		(pts
-			(xy 116.84 106.68) (xy 139.7 106.68)
-		)
-		(stroke
-			(width 0)
-			(type default)
-		)
-	)
-	(wire
-		(pts
 			(xy 160.02 57.15) (xy 86.36 57.15)
 		)
@@
 	(wire
 		(pts
-			(xy 115.57 52.07) (xy 115.57 104.14)
-		)
-		(stroke
+			(xy 203.2 111.76) (xy 203.2 116.84)
+		)
+		(stroke
